File: Actuator_Control.kicad_sch (KiCad schematic)
At the start: 15 parts, among them J15 Conn_01x02, J16 Conn_01x02, J17 Conn_01x02, Q5 BSS138, Q6 BSS138, Q7 BSS138

Commit message: Updated most of root-page labels.
Connections:
- net Nitrogen_Line_Control renamed Nitrous_Line_Control
Changed lines of the file:
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@@
 		)
 	)
-	(hierarchical_label "Nitrogen_Line_Control"
+	(hierarchical_label "Nitrous_Line_Control"
 		(shape input)
 		(at 203.2 87.63 180)

Commit message: Updated to 4-pin fans, moved power pages together, deleted old reference.
Parts:
- J4: renamed from J15; footprint Connector_Molex:Molex_Micro-Fit_3.0_43650-0215_1x02_P3.00mm_Vertical -> Connector_JST:JST_EH_B2B-EH-A_1x02_P2.50mm_Vertical
- J5: renamed from J16; footprint Connector_Molex:Molex_Micro-Fit_3.0_43650-0215_1x02_P3.00mm_Vertical -> Connector_JST:JST_EH_B2B-EH-A_1x02_P2.50mm_Vertical
- J6: renamed from J17; footprint Connector_Molex:Molex_Micro-Fit_3.0_43650-0215_1x02_P3.00mm_Vertical -> Connector_JST:JST_EH_B2B-EH-A_1x02_P2.50mm_Vertical
- renumbered D24 to D18, D25 to D19, D26 to D20, Q7 to Q3, Q5 to Q4, Q6 to Q5, R82 to R36, R84 to R37, R52 to R38, R53 to R39, R54 to R40, R55 to R41
Changed lines of the file:
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@@
 		(dnp no)
 		(fields_autoplaced yes)
-		(property "Reference" "J16"
+		(property "Reference" "J5"
 			(at 162.56 76.1999 0)
 			(effects
@@
 			)
 		)
-		(property "Footprint" "Connector_Molex:Molex_Micro-Fit_3.0_43650-0215_1x02_P3.00mm_Vertical"
+		(property "Footprint" "Connector_JST:JST_EH_B2B-EH-A_1x02_P2.50mm_Vertical"
 			(at 160.02 76.2 0)
 			(effects
@@
 			(project "QRET-ESP32"
 				(path "/24817451-dfe0-4b9a-9d93-7304529c9d58/6a16d2ee-e303-4211-9829-9eeec2519e33"
-					(reference "J16")
+					(reference "J5")
 					(unit 1)
 				)
@@
 		(dnp no)
 		(fields_autoplaced yes)
-		(property "Reference" "D24"
+		(property "Reference" "D18"
 			(at 75.946 72.39 0)
 			(effects
@@
 			(project "QRET-ESP32"
 				(path "/24817451-dfe0-4b9a-9d93-7304529c9d58/6a16d2ee-e303-4211-9829-9eeec2519e33"
-					(reference "D24")
+					(reference "D18")
 					(unit 1)
 				)
@@
 		(dnp no)
 		(fields_autoplaced yes)
-		(property "Reference" "#PWR095"
+		(property "Reference" "#PWR0189"
 			(at 228.6 78.74 0)
 			(effects
@@
 			(project "QRET-ESP32"
 				(path "/24817451-dfe0-4b9a-9d93-7304529c9d58/6a16d2ee-e303-4211-9829-9eeec2519e33"
-					(reference "#PWR095")
+					(reference "#PWR0189")
 					(unit 1)
 				)
@@
 		(dnp no)
 		(fields_autoplaced yes)
-		(property "Reference" "R84"
+		(property "Reference" "R37"
 			(at 71.12 88.8999 0)
 			(effects
@@
 			(project "QRET-ESP32"
 				(path "/24817451-dfe0-4b9a-9d93-7304529c9d58/6a16d2ee-e303-4211-9829-9eeec2519e33"
-					(reference "R84")
+					(reference "R37")
 					(unit 1)
 				)
@@
 		(dnp no)
 		(fields_autoplaced yes)
-		(property "Reference" "#PWR0171"
+		(property "Reference" "#PWR0195"
 			(at 68.58 80.01 0)
 			(effects
@@
 			(project "QRET-ESP32"
 				(path "/24817451-dfe0-4b9a-9d93-7304529c9d58/6a16d2ee-e303-4211-9829-9eeec2519e33"
-					(reference "#PWR0171")
+					(reference "#PWR0195")
 					(unit 1)
 				)
@@
 		(dnp no)
 		(fields_autoplaced yes)
-		(property "Reference" "Q6"
+		(property "Reference" "Q5"
 			(at 232.41 83.8199 0)
 			(effects
@@
 			(project "QRET-ESP32"
 				(path "/24817451-dfe0-4b9a-9d93-7304529c9d58/6a16d2ee-e303-4211-9829-9eeec2519e33"
-					(reference "Q6")
+					(reference "Q5")
 					(unit 1)
 				)
@@
 		(on_board yes)
 		(dnp no)
-		(property "Reference" "#PWR0172"
+		(property "Reference" "#PWR0198"
 			(at 68.58 99.06 0)
 			(effects
@@
 			(project "QRET-ESP32"
 				(path "/24817451-dfe0-4b9a-9d93-7304529c9d58/6a16d2ee-e303-4211-9829-9eeec2519e33"
-					(reference "#PWR0172")
+					(reference "#PWR0198")
 					(unit 1)
 				)
@@
 		(on_board yes)
 		(dnp no)
-		(property "Reference" "#PWR092"
+		(property "Reference" "#PWR0190"
 			(at 154.94 99.06 0)
 			(effects
@@
 			(project "QRET-ESP32"
 				(path "/24817451-dfe0-4b9a-9d93-7304529c9d58/6a16d2ee-e303-4211-9829-9eeec2519e33"
-					(reference "#PWR092")
+					(reference "#PWR0190")
 					(unit 1)
 				)
@@
 		(dnp no)
 		(fields_autoplaced yes)
-		(property "Reference" "D26"
+		(property "Reference" "D20"
 			(at 220.726 72.39 0)
 			(effects
@@
 			(project "QRET-ESP32"
 				(path "/24817451-dfe0-4b9a-9d93-7304529c9d58/6a16d2ee-e303-4211-9829-9eeec2519e33"
-					(reference "D26")
+					(reference "D20")
 					(unit 1)
 				)
@@
 		(on_board yes)
 		(dnp no)
-		(property "Reference" "#PWR096"
+		(property "Reference" "#PWR0192"
 			(at 228.6 99.06 0)
 			(effects
@@
 			(project "QRET-ESP32"
 				(path "/24817451-dfe0-4b9a-9d93-7304529c9d58/6a16d2ee-e303-4211-9829-9eeec2519e33"
-					(reference "#PWR096")
+					(reference "#PWR0192")
 					(unit 1)
 				)
@@
 		(dnp no)
 		(fields_autoplaced yes)
-		(property "Reference" "D25"
+		(property "Reference" "D19"
 			(at 147.066 72.39 0)
 			(effects
@@
 			(project "QRET-ESP32"
 				(path "/24817451-dfe0-4b9a-9d93-7304529c9d58/6a16d2ee-e303-4211-9829-9eeec2519e33"
-					(reference "D25")
+					(reference "D19")
 					(unit 1)
 				)
@@
 		(dnp no)
 		(fields_autoplaced yes)
-		(property "Reference" "#PWR0174"
+		(property "Reference" "#PWR0196"
 			(at 83.82 78.74 0)
 			(effects
@@
 			(project "QRET-ESP32"
 				(path "/24817451-dfe0-4b9a-9d93-7304529c9d58/6a16d2ee-e303-4211-9829-9eeec2519e33"
-					(reference "#PWR0174")
+					(reference "#PWR0196")
 					(unit 1)
 				)
@@
 		(dnp no)
 		(fields_autoplaced yes)
-		(property "Reference" "R53"
+		(property "Reference" "R39"
 			(at 142.24 88.8999 0)
 			(effects
@@
 			(project "QRET-ESP32"
 				(path "/24817451-dfe0-4b9a-9d93-7304529c9d58/6a16d2ee-e303-4211-9829-9eeec2519e33"
-					(reference "R53")
+					(reference "R39")
 					(unit 1)
 				)
@@
 		(dnp no)
 		(fields_autoplaced yes)
-		(property "Reference" "R52"
+		(property "Reference" "R38"
 			(at 133.35 81.28 90)
 			(effects
@@
 			(project "QRET-ESP32"
 				(path "/24817451-dfe0-4b9a-9d93-7304529c9d58/6a16d2ee-e303-4211-9829-9eeec2519e33"
-					(reference "R52")
+					(reference "R38")
 					(unit 1)
 				)
@@
 		(dnp no)
 		(fields_autoplaced yes)
-		(property "Reference" "J17"
+		(property "Reference" "J6"
 			(at 236.22 76.1999 0)
 			(effects
@@
 			)
 		)
-		(property "Footprint" "Connector_Molex:Molex_Micro-Fit_3.0_43650-0215_1x02_P3.00mm_Vertical"
+		(property "Footprint" "Connector_JST:JST_EH_B2B-EH-A_1x02_P2.50mm_Vertical"
 			(at 233.68 76.2 0)
 			(effects
@@
 			(project "QRET-ESP32"
 				(path "/24817451-dfe0-4b9a-9d93-7304529c9d58/6a16d2ee-e303-4211-9829-9eeec2519e33"
-					(reference "J17")
+					(reference "J6")
 					(unit 1)
 				)
@@
 		(dnp no)
 		(fields_autoplaced yes)
-		(property "Reference" "R54"
+		(property "Reference" "R40"
 			(at 207.01 81.28 90)
 			(effects
@@
 			(project "QRET-ESP32"
 				(path "/24817451-dfe0-4b9a-9d93-7304529c9d58/6a16d2ee-e303-4211-9829-9eeec2519e33"
-					(reference "R54")
+					(reference "R40")
 					(unit 1)
 				)
@@
 		(dnp no)
 		(fields_autoplaced yes)
-		(property "Reference" "Q7"
+		(property "Reference" "Q3"
 			(at 87.63 83.8199 0)
 			(effects
@@
 			(project "QRET-ESP32"
 				(path "/24817451-dfe0-4b9a-9d93-7304529c9d58/6a16d2ee-e303-4211-9829-9eeec2519e33"
-					(reference "Q7")
+					(reference "Q3")
 					(unit 1)
 				)
@@
 		(dnp no)
 		(fields_autoplaced yes)
-		(property "Reference" "#PWR091"
+		(property "Reference" "#PWR0191"
 			(at 154.94 78.74 0)
 			(effects
@@
 			(project "QRET-ESP32"
 				(path "/24817451-dfe0-4b9a-9d93-7304529c9d58/6a16d2ee-e303-4211-9829-9eeec2519e33"
-					(reference "#PWR091")
+					(reference "#PWR0191")
 					(unit 1)
 				)
@@
 		(on_board yes)
 		(dnp no)
-		(property "Reference" "#PWR090"
+		(property "Reference" "#PWR0194"
 			(at 139.7 99.06 0)
 			(effects
@@
 			(project "QRET-ESP32"
 				(path "/24817451-dfe0-4b9a-9d93-7304529c9d58/6a16d2ee-e303-4211-9829-9eeec2519e33"
-					(reference "#PWR090")
+					(reference "#PWR0194")
 					(unit 1)
 				)
@@
 		(dnp no)
 		(fields_autoplaced yes)
-		(property "Reference" "J15"
+		(property "Reference" "J4"
 			(at 91.44 76.1999 0)
 			(effects
@@
 			)
 		)
-		(property "Footprint" "Connector_Molex:Molex_Micro-Fit_3.0_43650-0215_1x02_P3.00mm_Vertical"
+		(property "Footprint" "Connector_JST:JST_EH_B2B-EH-A_1x02_P2.50mm_Vertical"
 			(at 88.9 76.2 0)
 			(effects
@@
 			(project "QRET-ESP32"
 				(path "/24817451-dfe0-4b9a-9d93-7304529c9d58/6a16d2ee-e303-4211-9829-9eeec2519e33"
-					(reference "J15")
+					(reference "J4")
 					(unit 1)
 				)
@@
 		(dnp no)
 		(fields_autoplaced yes)
-		(property "Reference" "R82"
+		(property "Reference" "R36"
 			(at 62.23 81.28 90)
 			(effects
@@
 			(project "QRET-ESP32"
 				(path "/24817451-dfe0-4b9a-9d93-7304529c9d58/6a16d2ee-e303-4211-9829-9eeec2519e33"
-					(reference "R82")
+					(reference "R36")
 					(unit 1)
 				)
@@
 		(dnp no)
 		(fields_autoplaced yes)
-		(property "Reference" "#PWR089"
+		(property "Reference" "#PWR0197"
 			(at 139.7 80.01 0)
 			(effects
@@
 			(project "QRET-ESP32"
 				(path "/24817451-dfe0-4b9a-9d93-7304529c9d58/6a16d2ee-e303-4211-9829-9eeec2519e33"
-					(reference "#PWR089")
+					(reference "#PWR0197")
 					(unit 1)
 				)
@@
 		(on_board yes)
 		(dnp no)
-		(property "Reference" "#PWR094"
+		(property "Reference" "#PWR0193"
 			(at 213.36 99.06 0)
 			(effects
@@
 			(project "QRET-ESP32"
 				(path "/24817451-dfe0-4b9a-9d93-7304529c9d58/6a16d2ee-e303-4211-9829-9eeec2519e33"
-					(reference "#PWR094")
+					(reference "#PWR0193")
 					(unit 1)
 				)
@@
 		(dnp no)
 		(fields_autoplaced yes)
-		(property "Reference" "Q5"
+		(property "Reference" "Q4"
 			(at 158.75 83.8199 0)
 			(effects
@@
 			(project "QRET-ESP32"
 				(path "/24817451-dfe0-4b9a-9d93-7304529c9d58/6a16d2ee-e303-4211-9829-9eeec2519e33"
-					(reference "Q5")
+					(reference "Q4")
 					(unit 1)
 				)
@@
 		(on_board yes)
 		(dnp no)
-		(property "Reference" "#PWR0175"
+		(property "Reference" "#PWR0199"
 			(at 83.82 99.06 0)
 			(effects
@@
 			(project "QRET-ESP32"
 				(path "/24817451-dfe0-4b9a-9d93-7304529c9d58/6a16d2ee-e303-4211-9829-9eeec2519e33"
-					(reference "#PWR0175")
+					(reference "#PWR0199")
 					(unit 1)
 				)
@@
 		(dnp no)
 		(fields_autoplaced yes)
-		(property "Reference" "R55"
+		(property "Reference" "R41"
 			(at 215.9 88.8999 0)
 			(effects
@@
 			(project "QRET-ESP32"
 				(path "/24817451-dfe0-4b9a-9d93-7304529c9d58/6a16d2ee-e303-4211-9829-9eeec2519e33"
-					(reference "R55")
+					(reference "R41")
 					(unit 1)
 				)
@@
 		(dnp no)
 		(fields_autoplaced yes)
-		(property "Reference" "#PWR093"
+		(property "Reference" "#PWR0188"
 			(at 213.36 80.01 0)
 			(effects
@@
 			(project "QRET-ESP32"
 				(path "/24817451-dfe0-4b9a-9d93-7304529c9d58/6a16d2ee-e303-4211-9829-9eeec2519e33"
-					(reference "#PWR093")
+					(reference "#PWR0188")
 					(unit 1)
 				)
