File: Control_Heating.kicad_sch (KiCad schematic)
At the start: 2 parts, among them J18 Conn_02x04_Counter_Clockwise, J19 Conn_02x04_Counter_Clockwise

Commit message: Added 24V-12V step-down converter for fans, started switch to devkit.
Other:
- note added: "System_Variable doesn't need to be ADCed."
Changed lines of the file:
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@@
+		)
+	)
+	(text "System_Variable doesn't need to be ADCed."
+		(exclude_from_sim no)
+		(at 67.818 84.328 0)
+		(effects
+			(font
+				(size 1.27 1.27)
+			)
 		)
 	)

Commit message: Updated to 4-pin fans, moved power pages together, deleted old reference.
Parts:
- J7: renamed from J19; footprint (none) -> Connector_JST:JST_J2100_B08B-J21DK-GGXR_2x04_P2.50x4.00mm_Vertical
- J8: renamed from J18; footprint (none) -> Connector_JST:JST_J2100_B08B-J21DK-GGXR_2x04_P2.50x4.00mm_Vertical
Changed lines of the file:
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@@
 		(dnp no)
 		(fields_autoplaced yes)
-		(property "Reference" "J19"
+		(property "Reference" "J7"
 			(at 74.93 87.63 0)
 			(effects
@@
 			)
 		)
-		(property "Footprint" ""
+		(property "Footprint" "Connector_JST:JST_J2100_B08B-J21DK-GGXR_2x04_P2.50x4.00mm_Vertical"
 			(at 73.66 96.52 0)
 			(effects
@@
 			(project ""
 				(path "/24817451-dfe0-4b9a-9d93-7304529c9d58/0c734fb5-09c2-4b1e-989d-a08b4d481f06"
-					(reference "J19")
+					(reference "J7")
 					(unit 1)
 				)
@@
 		(dnp no)
 		(fields_autoplaced yes)
-		(property "Reference" "J18"
+		(property "Reference" "J8"
 			(at 138.43 87.63 0)
 			(effects
@@
 			)
 		)
-		(property "Footprint" ""
+		(property "Footprint" "Connector_JST:JST_J2100_B08B-J21DK-GGXR_2x04_P2.50x4.00mm_Vertical"
 			(at 137.16 96.52 0)
 			(effects
@@
 			(project "QRET-ESP32"
 				(path "/24817451-dfe0-4b9a-9d93-7304529c9d58/0c734fb5-09c2-4b1e-989d-a08b4d481f06"
-					(reference "J18")
+					(reference "J8")
 					(unit 1)
 				)
